Commit message: Add dynamic TCP

File: e2f_description/urdf/e2f.ros2_control.xacro (robot description, xacro)
@@ -47,4 +47,9 @@
         </state_interface>
       </joint>
+      <joint name="${tf_prefix}tcp_joint">
+        <state_interface name="position">
+          <param name="initial_value">0.13</param>
+        </state_interface>
+      </joint>
       <xacro:unless value="${use_fake_hardware}">
         <gpio name="${tf_prefix}stroke">

File: e2f_description/urdf/e2f_macro.xacro (robot description, xacro)
@@ -193,4 +193,13 @@
       <origin xyz="8e-3 0 17e-3" rpy="0 0 0" />
     </joint>
+    <!-- TCP -->
+    <link name="${tf_prefix}tcp" />
+    <joint name="${tf_prefix}tcp_joint" type="prismatic">
+      <parent link="${tf_prefix}base_link" />
+      <child link="${tf_prefix}tcp" />
+      <origin xyz="0 0 0" rpy="0 0 0" />
+      <axis xyz="0 0 1" />
+      <limit upper="0" lower="0.2" effort="0" velocity="0" />
+    </joint>
   </xacro:macro>
 </robot>

Commit message: Use joint element for stroke interface to publish state value via joint_state_broadcaster

File: e2f_description/urdf/e2f.ros2_control.xacro (robot description, xacro)
@@ -52,11 +52,13 @@
         </state_interface>
       </joint>
-      <xacro:unless value="${use_fake_hardware}">
-        <gpio name="${tf_prefix}stroke">
-          <command_interface name="width" />
-          <state_interface name="width" />
-          <state_interface name="force" />
-        </gpio>
-      </xacro:unless>
+      <joint name="${tf_prefix}stroke">
+        <command_interface name="position" />
+        <state_interface name="position">
+          <param name="initial_value">0.0</param>
+        </state_interface>
+        <state_interface name="effort">
+          <param name="initial_value">0.0</param>
+        </state_interface>
+      </joint>
     </ros2_control>
   </xacro:macro>

File: e2f_description/urdf/e2f_macro.xacro (robot description, xacro)
@@ -193,4 +193,13 @@
       <origin xyz="8e-3 0 17e-3" rpy="0 0 0" />
     </joint>
+    <!-- Stroke -->
+    <link name="${tf_prefix}stroke_end" />
+    <joint name="${tf_prefix}stroke" type="prismatic">
+      <parent link="${tf_prefix}fingertip_r" />
+      <child link="${tf_prefix}stroke_end" />
+      <origin xyz="0 0 0" rpy="0 0 0" />
+      <axis xyz="1 0 0" />
+      <limit upper="0" lower="0" effort="0" velocity="0" />
+    </joint>
     <!-- TCP -->
     <link name="${tf_prefix}tcp" />
