Commit message: Remove gear visuals

File: e2f_description/urdf/e2f_macro.xacro (robot description, xacro)
@@ -39,18 +39,6 @@
       </collision>
     </link>
-    <link name="${tf_prefix}gear_l">
-      <visual>
-        <geometry>
-          <mesh filename="file://${description_package}/meshes/visual/gear_l.dae" />
-        </geometry>
-      </visual>
-    </link>
-    <link name="${tf_prefix}gear_r">
-      <visual>
-        <geometry>
-          <mesh filename="file://${description_package}/meshes/visual/gear_r.dae" />
-        </geometry>
-      </visual>
-    </link>
+    <link name="${tf_prefix}gear_l" />
+    <link name="${tf_prefix}gear_r" />
     <link name="${tf_prefix}link1_l">
       <visual>

Commit message: Fix joint limits

File: e2f_description/urdf/e2f_macro.xacro (robot description, xacro)
@@ -188,5 +188,5 @@
       <origin xyz="0 0 0" rpy="0 0 0" />
       <axis xyz="1 0 0" />
-      <limit upper="0" lower="0" effort="0" velocity="0" />
+      <limit upper="1.0" lower="-1.0" effort="1.0" velocity="1.0" />
     </joint>
     <!-- TCP -->
@@ -197,5 +197,5 @@
       <origin xyz="0 0 0" rpy="0 0 0" />
       <axis xyz="0 0 1" />
-      <limit upper="0" lower="0.2" effort="0" velocity="0" />
+      <limit upper="1.0" lower="0" effort="1.0" velocity="1.0" />
     </joint>
   </xacro:macro>
